File: hardware/Transistor_Driver.kicad_sch (KiCad schematic)
At the start: 11 parts, among them J1 Conn_GND, J2 Power_Output, J3 Conn_5V, K2 G5LE-1, Q2 BC547

Commit message: feat(hardware): add PCB design
Parts:
- renumbered D3 to D1, J3 to J1, J1 to J2, J2 to J3, K2 to K1, Q2 to Q1, R3 to R1, R1 to R2, R2 to R3
Changed lines of the file:
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@@
 		(dnp no)
 		(fields_autoplaced yes)
-		(property "Reference" "#PWR02"
+		(property "Reference" "#PWR04"
 			(at 95.25 91.44 0)
 			(hide yes)
@@
 			(project "Transistor_Driver"
 				(path "/3229a635-ec2b-40b4-9555-10d0ea3caa11"
-					(reference "#PWR02")
+					(reference "#PWR04")
 					(unit 1)
 				)
@@
 		(dnp no)
 		(fields_autoplaced yes)
-		(property "Reference" "R3"
+		(property "Reference" "R1"
 			(at 59.69 74.9299 0)
 			(show_name no)
@@
 			(project "Transistor_Driver"
 				(path "/3229a635-ec2b-40b4-9555-10d0ea3caa11"
-					(reference "R3")
+					(reference "R1")
 					(unit 1)
 				)
@@
 		(dnp no)
 		(fields_autoplaced yes)
-		(property "Reference" "J1"
+		(property "Reference" "J2"
 			(at 48.26 41.9099 0)
 			(show_name no)
@@
 			(project "Transistor_Driver"
 				(path "/3229a635-ec2b-40b4-9555-10d0ea3caa11"
-					(reference "J1")
+					(reference "J2")
 					(unit 1)
 				)
@@
 		(dnp no)
 		(fields_autoplaced yes)
-		(property "Reference" "Q2"
+		(property "Reference" "Q1"
 			(at 97.79 68.5799 0)
 			(show_name no)
@@
 			(project "Transistor_Driver"
 				(path "/3229a635-ec2b-40b4-9555-10d0ea3caa11"
-					(reference "Q2")
+					(reference "Q1")
 					(unit 1)
 				)
@@
 		(dnp no)
 		(fields_autoplaced yes)
-		(property "Reference" "J3"
+		(property "Reference" "J1"
 			(at 48.26 35.5599 0)
 			(show_name no)
@@
 			(project "Transistor_Driver"
 				(path "/3229a635-ec2b-40b4-9555-10d0ea3caa11"
-					(reference "J3")
+					(reference "J1")
 					(unit 1)
 				)
@@
 		(dnp no)
 		(fields_autoplaced yes)
-		(property "Reference" "K2"
+		(property "Reference" "K1"
 			(at 111.76 38.0999 0)
 			(show_name no)
@@
 			(project "Transistor_Driver"
 				(path "/3229a635-ec2b-40b4-9555-10d0ea3caa11"
-					(reference "K2")
+					(reference "K1")
 					(unit 1)
 				)
@@
 		(dnp no)
 		(fields_autoplaced yes)
-		(property "Reference" "D3"
+		(property "Reference" "D1"
 			(at 78.74 39.3699 90)
 			(show_name no)
@@
 			(project "Transistor_Driver"
 				(path "/3229a635-ec2b-40b4-9555-10d0ea3caa11"
-					(reference "D3")
+					(reference "D1")
 					(unit 1)
 				)
@@
 		(dnp no)
 		(fields_autoplaced yes)
-		(property "Reference" "R1"
+		(property "Reference" "R2"
 			(at 71.12 63.5 90)
 			(show_name no)
@@
 			(project "Transistor_Driver"
 				(path "/3229a635-ec2b-40b4-9555-10d0ea3caa11"
-					(reference "R1")
+					(reference "R2")
 					(unit 1)
 				)
@@
 		(dnp no)
 		(fields_autoplaced yes)
-		(property "Reference" "#PWR03"
+		(property "Reference" "#PWR02"
 			(at 31.75 39.37 0)
 			(hide yes)
@@
 			(project "Transistor_Driver"
 				(path "/3229a635-ec2b-40b4-9555-10d0ea3caa11"
-					(reference "#PWR03")
+					(reference "#PWR02")
 					(unit 1)
 				)
@@
 		(dnp no)
 		(fields_autoplaced yes)
-		(property "Reference" "R2"
+		(property "Reference" "R3"
 			(at 125.73 68.5799 0)
 			(show_name no)
@@
 			(project "Transistor_Driver"
 				(path "/3229a635-ec2b-40b4-9555-10d0ea3caa11"
-					(reference "R2")
+					(reference "R3")
 					(unit 1)
 				)
@@
 		(dnp no)
 		(fields_autoplaced yes)
-		(property "Reference" "#PWR04"
+		(property "Reference" "#PWR03"
 			(at 31.75 50.8 0)
 			(hide yes)
@@
 			(project "Transistor_Driver"
 				(path "/3229a635-ec2b-40b4-9555-10d0ea3caa11"
-					(reference "#PWR04")
+					(reference "#PWR03")
 					(unit 1)
 				)
@@
 		(dnp no)
 		(fields_autoplaced yes)
-		(property "Reference" "J2"
+		(property "Reference" "J3"
 			(at 151.13 66.0399 0)
 			(show_name no)
@@
 			(project "Transistor_Driver"
 				(path "/3229a635-ec2b-40b4-9555-10d0ea3caa11"
-					(reference "J2")
-					(unit 1)
-				)
+					(reference "J3")
+					(unit 1)
+				)
