File: hardware/PCB/Transistor_Driver.kicad_sch (KiCad schematic)
At the start: 11 parts, among them J1 Conn_5V, J2 Conn_GND, J3 Power_Output, K1 G5LE-1, Q1 BC547

Commit message: feat(hardware): release v1r2
Parts:
- D1: footprint Diode_THT:D_DO-201AD_P15.24mm_Horizontal -> Transistor_Driver-Footprints:D_DO-201AD_P15.24mm_Horizontal
- D2: footprint LED_THT:LED_D3.0mm -> Transistor_Driver-Footprints:LED_D3.0mm_Clear
- J1, J2: footprint Connector_PinHeader_2.54mm:PinHeader_1x01_P2.54mm_Vertical -> Transistor_Driver-Footprints:PinHeader_1x01_P2.54mm_Vertical
- J3: footprint TerminalBlock_Phoenix:TerminalBlock_Phoenix_PT-1,5-2-5.0-H_1x02_P5.00mm_Horizontal -> Transistor_Driver-Footprints:TerminalBlock_Phoenix_PT-1,5-2-5.0-H_1x02_P5.00mm_Horizontal
- K1: footprint Relay_THT:Relay_SPDT_Omron-G5LE-1 -> Transistor_Driver-Footprints:Relay_SPDT_Omron-G5LE-1
- Q1: footprint Package_TO_SOT_THT:TO-92_Inline -> Transistor_Driver-Footprints:TO-92_Inline_Wide
- R1, R2, R3: footprint Resistor_THT:R_Axial_DIN0207_L6.3mm_D2.5mm_P10.16mm_Horizontal -> Transistor_Driver-Footprints:R_Axial_DIN0207_L6.3mm_D2.5mm_P10.16mm_Horizontal
- S1: footprint PS1024ALRED:SW_PS1024ALRED -> Transistor_Driver-Footprints:SW_PS1024ALRED
Changed lines of the file:
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@@
 			)
 		)
-		(property "Footprint" "LED_THT:LED_D3.0mm"
+		(property "Footprint" "Transistor_Driver-Footprints:LED_D3.0mm_Clear"
 			(at 123.19 57.15 0)
 			(hide yes)
@@
 			)
 		)
-		(property "Footprint" "Resistor_THT:R_Axial_DIN0207_L6.3mm_D2.5mm_P10.16mm_Horizontal"
+		(property "Footprint" "Transistor_Driver-Footprints:R_Axial_DIN0207_L6.3mm_D2.5mm_P10.16mm_Horizontal"
 			(at 55.372 76.2 90)
 			(hide yes)
@@
 			)
 		)
-		(property "Footprint" "Connector_PinHeader_2.54mm:PinHeader_1x01_P2.54mm_Vertical"
+		(property "Footprint" "Transistor_Driver-Footprints:PinHeader_1x01_P2.54mm_Vertical"
 			(at 45.72 43.18 0)
 			(hide yes)
@@
 			)
 		)
-		(property "Footprint" "Package_TO_SOT_THT:TO-92_Inline"
+		(property "Footprint" "Transistor_Driver-Footprints:TO-92_Inline_Wide"
 			(at 97.79 71.755 0)
 			(hide yes)
@@
 			)
 		)
-		(property "Footprint" "Connector_PinHeader_2.54mm:PinHeader_1x01_P2.54mm_Vertical"
+		(property "Footprint" "Transistor_Driver-Footprints:PinHeader_1x01_P2.54mm_Vertical"
 			(at 45.72 36.83 0)
 			(hide yes)
@@
 			)
 		)
-		(property "Footprint" "PS1024ALRED:SW_PS1024ALRED"
+		(property "Footprint" "Transistor_Driver-Footprints:SW_PS1024ALRED"
 			(at 43.18 69.85 0)
 			(hide yes)
@@
 			)
 		)
-		(property "Footprint" "Relay_THT:Relay_SPDT_Omron-G5LE-1"
+		(property "Footprint" "Transistor_Driver-Footprints:Relay_SPDT_Omron-G5LE-1"
 			(at 111.76 40.64 0)
 			(hide yes)
@@
 			)
 		)
-		(property "Footprint" "Diode_THT:D_DO-201AD_P15.24mm_Horizontal"
+		(property "Footprint" "Transistor_Driver-Footprints:D_DO-201AD_P15.24mm_Horizontal"
 			(at 71.755 40.64 0)
 			(hide yes)
@@
 			)
 		)
-		(property "Footprint" "Resistor_THT:R_Axial_DIN0207_L6.3mm_D2.5mm_P10.16mm_Horizontal"
+		(property "Footprint" "Transistor_Driver-Footprints:R_Axial_DIN0207_L6.3mm_D2.5mm_P10.16mm_Horizontal"
 			(at 71.12 71.628 90)
 			(hide yes)
@@
 			)
 		)
-		(property "Footprint" "Resistor_THT:R_Axial_DIN0207_L6.3mm_D2.5mm_P10.16mm_Horizontal"
+		(property "Footprint" "Transistor_Driver-Footprints:R_Axial_DIN0207_L6.3mm_D2.5mm_P10.16mm_Horizontal"
 			(at 124.968 69.85 90)
 			(hide yes)
@@
 			)
 		)
-		(property "Footprint" "TerminalBlock_Phoenix:TerminalBlock_Phoenix_PT-1,5-2-5.0-H_1x02_P5.00mm_Horizontal"
+		(property "Footprint" "Transistor_Driver-Footprints:TerminalBlock_Phoenix_PT-1,5-2-5.0-H_1x02_P5.00mm_Horizontal"
 			(at 148.59 66.04 0)
 			(hide yes)
